File: KiCad/F800_arduino_v1.kicad_sch (KiCad schematic)
At the start: 50 parts, among them U1 L7808, U1 PC817

Commit message: Update dtmf
Parts:
- removed C?: 150nF, symbol Device:C_Small
- removed JP1, JP?: (no value), symbol Device:Jumper_NC_Small
- removed R?: 22k, symbol Device:R_Small
- added C?: 22uF, symbol Device:C_Small
- added D? (x2): 1N4001, Diode_THT:D_DO-41_SOD81_P10.16mm_Horizontal, symbol Diode:1N4001
- added R? (x3): 1k, symbol Device:R_Small
- added R? (x2): 10k, symbol Device:R_Small
- added R?: 22k, symbol Device:R_Small
Connections:
- net +5V: now also D?.1 (K), R?.1
- net GND: now also D?.2 (A), R?.2
- net at A1.19 (A0): now also D?.1 (K), D?.2 (A), R?.1, R?.2, R?.2, R?.2
- net at A1.5 (D2), R?.2: now also R?.2
- net at ..10 (Pin_10): now also ..9 (Pin_9)
- net at ..2 (Pin_2): now also C?.2
- net at ..4 (Pin_4): now also R?.1
- net at ..5 (Pin_5): now also C?.2, R?.1
- net at R?.1, U?.14: now also R?.1
- net at C?.1: now also R?.2
- new net: C?.1, R?.1, R?.1
Other:
- note added: "DTMF in"
- note removed: "Sound bypass"
- title: ctcss and scanning for Ericsson F800  -> ctcss, dtmf and scanning for Ericsson F800 
